File: KiCad/Delta.kicad_pcb (KiCad board)
At the start: 2 copper layers, 156.9 x 147.6 mm, 41 parts, among them J1 Conn_01x03, J2 Conn_01x05, J3 MAC-22, Q151 2SD468, Q152 D44C8, U1 74LVC1G04

Commit message: Add files via upload
Parts:
- removed the G*** at (186.2, 139.6)
- added G***: LOGO, LOGO, F.Cu at (202.0, 134.8)
- added G***: LOGO, LOGO, F.Cu at (150.8, 98.1)
- added REF**: Symbol_HighVoltage_Triangle_8x7mm_Copper, Symbol:Symbol_HighVoltage_Triangle_8x7mm_Copper, F.Cu at (140.2, 137.6)
- added REF**: Symbol_HighVoltage_Triangle_8x7mm_Copper, Symbol:Symbol_HighVoltage_Triangle_8x7mm_Copper, F.Cu at (186.3, 137.6)
- added REF**: Symbol_HighVoltage_Triangle_8x7mm_Copper, Symbol:Symbol_HighVoltage_Triangle_8x7mm_Copper, F.Cu at (183.1, 137.6)
- moved Q152 10.8 mm to (108.6, 134.8)
- moved PAD13 1.53 mm to (157.2, 135.9)
- moved PAD14 1.53 mm to (150.4, 135.9)
Routing:
- net Net-(J1-Pin_1): track 64.3 -> 57.0 mm, vias 1 -> 2
- net GND: track 649.6 -> 656.3 mm, vias 3 -> 4
- net Net-(Q151-E): track 55.2 -> 48.5 mm
- net Net-(J2-L-Pad2): track 49.3 -> 47.8 mm
- net Net-(J2-N-Pad4): track 41.7 -> 41.0 mm
Other:
- board text added: "ATX Conversion Board for Delta SMP-220DB V1.2"
- board text added: "ATX Conversion Board for Delta SMP-220DB V1.2 github.com/croissantking/840AV-Stealth-ATX"
- board text added: "CAUTION HIGH VOLTAGE"
- board text removed: "ATX Conversion Board V1.1 for Delta SMP-220DB github.com/croissantking"
